Commit message: update

File: src/cpp_wcl/model/robot_model.xacro (robot description, xacro)
@@ -31,11 +31,11 @@
   <!-- Over Here  we include the file that defines extra Gazebo options and motion control drivers -->
    <xacro:include filename="$(find cpp_wcl )/model/robot.gazebo"/>
-<link name="dummy">
+<!-- <link name="dummy">
 </link>
 <joint name="dummy_joint" type="fixed">
     <parent link="dummy"/>
-    <child link="body_link"/>
-</joint>
-<link name="body_link">
+    <child link="base_link"/>
+</joint> -->
+<link name="base_link">
     <visual>
         <geometry><box size="${body_link_x_dim} ${body_link_y_dim} ${body_link_z_dim}"/></geometry>
@@ -59,5 +59,5 @@
 <!-- Start : Back Right wheel -->
 <joint name="wheel1_joint" type="continuous">
-    <parent link="body_link"/>
+    <parent link="base_link"/>
     <child link="wheel1_link"/>
     <origin xyz="-0.3 -0.35 0.0" rpy="0 0 0"/>
@@ -82,5 +82,5 @@
     <!-- Start : Back left wheel -->
      <joint name="wheel2_joint" type="continuous">
-    <parent link="body_link"/>
+    <parent link="base_link"/>
     <child link="wheel2_link"/>
     <origin xyz="-0.3 0.35 0.0" rpy="0 0 0"/>
@@ -105,5 +105,5 @@
      <!-- Start : front right wheel_3 -->
 <joint name="wheel3_joint" type="continuous">
-    <parent link="body_link"/>
+    <parent link="base_link"/>
     <child link="wheel3_link"/>
     <origin xyz="0.3 -0.35 0.0" rpy="0 0 0"/>
@@ -128,5 +128,5 @@
      <!-- Start : front left wheel 4 -->
      <joint name="wheel4_joint" type="continuous">
-    <parent link="body_link"/>
+    <parent link="base_link"/>
     <child link="wheel4_link"/>
     <origin xyz="0.3 0.35 0.0" rpy="0 0 0"/>
@@ -150,11 +150,11 @@
     <!-- LIDAR-->
      <joint name="lidar_joint" type="fixed">
-        <origin xyz="0.3 0.0 0.1" rpy="0 0 0"/>
-        <parent link="body_link"/>
+        <origin xyz="0.3 0.0 0.25" rpy="0 0 0"/>
+        <parent link="base_link"/>
         <child link="lidar_link"/>
      </joint>
     <link name='lidar_link'>
         <visual>
-            <origin xyz="0 0 0.05" rpy="0 1.0 0 "/>
+            <origin xyz="0 0 0.05" rpy="0 0 0 "/>
             <geometry>
                 <cylinder radius="0.1" length="0.1"/>
@@ -177,5 +177,5 @@
     <joint name="imu_joint" type="fixed">
         <origin xyz="0 0 0" rpy="0 0 0"/>
-        <parent link="body_link"/>
+        <parent link="base_link"/>
         <child link="imu_link"/>
     </joint>
